File: WiredControllerPcb.sch (KiCad schematic (older format))
At the start: 33 parts, among them J1 Joystick, J2 Conn_01x06, J3 Conn_01x04, J4 Conn_01x04, SW1 SW_Push, SW2 SW_Push, SW3 SW_Push, SW4 SW_Push, U1 LP2985-3.3, U2 ATmega328P-MU

Commit message: Add pin header
Parts:
- added J5: Conn_01x04, Connector_PinHeader_2.54mm:PinHeader_1x04_P2.54mm_Vertical, symbol Connector_Generic:Conn_01x04
Connections:
- net GND: now also J5.4 (Pin_4)
- net SCL: now also J5.1 (Pin_1)
- net SDA: now also J5.2 (Pin_2)
- net VDC: now also J5.3 (Pin_3)
Changed lines of the file:
@@
 	1    0    0    -1
 $EndComp
-Text Label 9150 4300 0    50   ~ 0
-SDA
-Text Label 9150 4200 0    50   ~ 0
-SCL
+Wire Wire Line
+	9150 4400 9400 4400
 $Comp
 L power:VDC #PWR0122
@@
 	1    0    0    -1
 $EndComp
+Text Label 9150 4200 0    50   ~ 0
+SCL
+Text Label 9150 4300 0    50   ~ 0
+SDA
+$Comp
+L Connector_Generic:Conn_01x04 J5
+U 1 1 5D85B462
+P 8950 5150
+F 0 "J5" H 8868 5467 50  0000 C CNN
+F 1 "Conn_01x04" H 8868 5376 50  0000 C CNN
+F 2 "Connector_PinHeader_2.54mm:PinHeader_1x04_P2.54mm_Vertical" H 8950 5150 50  0001 C CNN
+F 3 "~" H 8950 5150 50  0001 C CNN
+	1    8950 5150
+	-1   0    0    -1
+$EndComp
+$Comp
+L power:GND #PWR0125
+U 1 1 5D85B468
+P 9150 5350
+F 0 "#PWR0125" H 9150 5100 50  0001 C CNN
+F 1 "GND" H 9155 5177 50  0000 C CNN
+F 2 "" H 9150 5350 50  0001 C CNN
+F 3 "" H 9150 5350 50  0001 C CNN
+	1    9150 5350
+	1    0    0    -1
+$EndComp
 Wire Wire Line
-	9150 4400 9400 4400
+	9150 5250 9400 5250
+$Comp
+L power:VDC #PWR0126
+U 1 1 5D85B46F
+P 9400 5250
+F 0 "#PWR0126" H 9400 5150 50  0001 C CNN
+F 1 "VDC" H 9400 5525 50  0000 C CNN
+F 2 "" H 9400 5250 50  0001 C CNN
+F 3 "" H 9400 5250 50  0001 C CNN
+	1    9400 5250
+	1    0    0    -1
+$EndComp
+Text Label 9150 5050 0    50   ~ 0
+SCL
+Text Label 9150 5150 0    50   ~ 0
+SDA
 $EndSCHEMATC

Commit message: Change resister to pullup to 10k from 1k
Parts:
- R7, R8: value 1k -> 10k
Changed lines of the file:
@@
 P 7850 3400
 F 0 "R7" V 7750 3400 50  0000 C CNN
-F 1 "1k" V 7850 3400 50  0000 C CNN
+F 1 "10k" V 7850 3400 50  0000 C CNN
 F 2 "Resistor_SMD:R_0603_1608Metric" V 7780 3400 50  0001 C CNN
 F 3 "~" H 7850 3400 50  0001 C CNN
@@
 P 7850 3700
 F 0 "R8" V 7750 3700 50  0000 C CNN
-F 1 "1k" V 7850 3700 50  0000 C CNN
+F 1 "10k" V 7850 3700 50  0000 C CNN
 F 2 "Resistor_SMD:R_0603_1608Metric" V 7780 3700 50  0001 C CNN
 F 3 "~" H 7850 3700 50  0001 C CNN

Commit message: Add pull up resistor to reset pin
Parts:
- added R9: 10k, Resistor_SMD:R_0603_1608Metric, symbol Device:R
- U2: symbol MCU_Microchip_ATmega:ATmega328P-MU -> WiredControllerPcb-rescue:ATmega328P-MU-MCU_Microchip_ATmega
Connections:
- net +3V3: now also R9.1
- net RST: now also R9.2
Changed lines of the file:
@@
 EESchema Schematic File Version 4
-LIBS:WiredControllerPcb-cache
 EELAYER 30 0
 EELAYER END
@@
 	2900 4250 2900 4050
 $Comp
-L MCU_Microchip_ATmega:ATmega328P-MU U2
+L WiredControllerPcb-rescue:ATmega328P-MU-MCU_Microchip_ATmega U2
 U 1 1 5D26AB1A
 P 5850 3800
@@
 Text Label 9150 5150 0    50   ~ 0
 SDA
+$Comp
+L Device:R R9
+U 1 1 5E407ED2
+P 7850 4050
+F 0 "R9" V 7750 4050 50  0000 C CNN
+F 1 "10k" V 7850 4050 50  0000 C CNN
+F 2 "Resistor_SMD:R_0603_1608Metric" V 7780 4050 50  0001 C CNN
+F 3 "~" H 7850 4050 50  0001 C CNN
+	1    7850 4050
+	0    1    1    0
+$EndComp
+Text Label 7700 4050 2    50   ~ 0
+RST
+Wire Wire Line
+	8000 4050 8050 4050
+Wire Wire Line
+	8050 4050 8050 3700
+Connection ~ 8050 3700
 $EndSCHEMATC
